File: Icicle.sch (KiCad schematic (older format))
At the start: 23 parts, among them P1 NeopixelStripPads, P2 NeopixelStripPads

Commit message: Added a by-pass cap
Parts:
- added C1: 10uF, Capacitor_SMD:C_1206_3216Metric, symbol Device:C
Connections:
- net +5V: now also C1.2
- net GND: now also C1.1
Changed lines of the file:
@@
 $EndComp
 Wire Wire Line
-	8500 1800 8500 1950
+	8500 1800 8500 1850
 $Comp
 L power:GND #PWR0102
@@
 $EndComp
 Wire Wire Line
-	8900 1800 8900 1950
+	8900 1800 8900 1850
 $Comp
 L Mechanical:MountingHole H1
@@
 	-1   0    0    1
 $EndComp
+$Comp
+L Device:C C1
+U 1 1 60272B9A
+P 8700 1850
+F 0 "C1" V 8952 1850 50  0000 C CNN
+F 1 "10uF" V 8861 1850 50  0000 C CNN
+F 2 "Capacitor_SMD:C_1206_3216Metric" H 8738 1700 50  0001 C CNN
+F 3 "~" H 8700 1850 50  0001 C CNN
+	1    8700 1850
+	0    1    -1   0
+$EndComp
+Wire Wire Line
+	8850 1850 8900 1850
+Connection ~ 8900 1850
+Wire Wire Line
+	8900 1850 8900 1950
+Wire Wire Line
+	8550 1850 8500 1850
+Connection ~ 8500 1850
+Wire Wire Line
+	8500 1850 8500 1950
 $EndSCHEMATC

Commit message: Added LCSC parts
Parts:
- C1: LCSC (none) -> C13585
- D1, D10, D11, D12, D13, D14, D15, D16, D17, D18, D19, D2, D20, D3, D4, D5, D6, D7, D8, D9: LCSC (none) -> C114586
Changed lines of the file:
@@
 F 2 "LED_SMD:LED_WS2812B_PLCC4_5.0x5.0mm_P3.2mm" H 1450 2150 50  0001 L TNN
 F 3 "https://cdn-shop.adafruit.com/datasheets/WS2812B.pdf" H 1500 2075 50  0001 L TNN
+F 4 "C114586" H 1400 2450 50  0001 C CNN "LCSC"
 	1    1400 2450
 	1    0    0    -1
@@
 F 2 "LED_SMD:LED_WS2812B_PLCC4_5.0x5.0mm_P3.2mm" H 2450 2150 50  0001 L TNN
 F 3 "https://cdn-shop.adafruit.com/datasheets/WS2812B.pdf" H 2500 2075 50  0001 L TNN
+F 4 "C114586" H 2400 2450 50  0001 C CNN "LCSC"
 	1    2400 2450
 	1    0    0    -1
@@
 F 2 "LED_SMD:LED_WS2812B_PLCC4_5.0x5.0mm_P3.2mm" H 4450 2150 50  0001 L TNN
 F 3 "https://cdn-shop.adafruit.com/datasheets/WS2812B.pdf" H 4500 2075 50  0001 L TNN
+F 4 "C114586" H 4400 2450 50  0001 C CNN "LCSC"
 	1    4400 2450
 	1    0    0    -1
@@
 F 2 "LED_SMD:LED_WS2812B_PLCC4_5.0x5.0mm_P3.2mm" H 3450 2150 50  0001 L TNN
 F 3 "https://cdn-shop.adafruit.com/datasheets/WS2812B.pdf" H 3500 2075 50  0001 L TNN
+F 4 "C114586" H 3400 2450 50  0001 C CNN "LCSC"
 	1    3400 2450
 	1    0    0    -1
@@
 F 2 "LED_SMD:LED_WS2812B_PLCC4_5.0x5.0mm_P3.2mm" H 5450 2150 50  0001 L TNN
 F 3 "https://cdn-shop.adafruit.com/datasheets/WS2812B.pdf" H 5500 2075 50  0001 L TNN
+F 4 "C114586" H 5400 2450 50  0001 C CNN "LCSC"
 	1    5400 2450
 	1    0    0    -1
@@
 F 2 "LED_SMD:LED_WS2812B_PLCC4_5.0x5.0mm_P3.2mm" H 1450 3450 50  0001 L TNN
 F 3 "https://cdn-shop.adafruit.com/datasheets/WS2812B.pdf" H 1500 3375 50  0001 L TNN
+F 4 "C114586" H 1400 3750 50  0001 C CNN "LCSC"
 	1    1400 3750
 	1    0    0    -1
@@
 F 2 "LED_SMD:LED_WS2812B_PLCC4_5.0x5.0mm_P3.2mm" H 2450 3450 50  0001 L TNN
 F 3 "https://cdn-shop.adafruit.com/datasheets/WS2812B.pdf" H 2500 3375 50  0001 L TNN
+F 4 "C114586" H 2400 3750 50  0001 C CNN "LCSC"
 	1    2400 3750
 	1    0    0    -1
@@
 F 2 "LED_SMD:LED_WS2812B_PLCC4_5.0x5.0mm_P3.2mm" H 4450 3450 50  0001 L TNN
 F 3 "https://cdn-shop.adafruit.com/datasheets/WS2812B.pdf" H 4500 3375 50  0001 L TNN
+F 4 "C114586" H 4400 3750 50  0001 C CNN "LCSC"
 	1    4400 3750
 	1    0    0    -1
@@
 F 2 "LED_SMD:LED_WS2812B_PLCC4_5.0x5.0mm_P3.2mm" H 3450 3450 50  0001 L TNN
 F 3 "https://cdn-shop.adafruit.com/datasheets/WS2812B.pdf" H 3500 3375 50  0001 L TNN
+F 4 "C114586" H 3400 3750 50  0001 C CNN "LCSC"
 	1    3400 3750
 	1    0    0    -1
@@
 F 2 "LED_SMD:LED_WS2812B_PLCC4_5.0x5.0mm_P3.2mm" H 5450 3450 50  0001 L TNN
 F 3 "https://cdn-shop.adafruit.com/datasheets/WS2812B.pdf" H 5500 3375 50  0001 L TNN
+F 4 "C114586" H 5400 3750 50  0001 C CNN "LCSC"
 	1    5400 3750
 	1    0    0    -1
@@
 F 2 "LED_SMD:LED_WS2812B_PLCC4_5.0x5.0mm_P3.2mm" H 1450 4750 50  0001 L TNN
 F 3 "https://cdn-shop.adafruit.com/datasheets/WS2812B.pdf" H 1500 4675 50  0001 L TNN
+F 4 "C114586" H 1400 5050 50  0001 C CNN "LCSC"
 	1    1400 5050
 	1    0    0    -1
@@
 F 2 "LED_SMD:LED_WS2812B_PLCC4_5.0x5.0mm_P3.2mm" H 2450 4750 50  0001 L TNN
 F 3 "https://cdn-shop.adafruit.com/datasheets/WS2812B.pdf" H 2500 4675 50  0001 L TNN
+F 4 "C114586" H 2400 5050 50  0001 C CNN "LCSC"
 	1    2400 5050
 	1    0    0    -1
@@
 F 2 "LED_SMD:LED_WS2812B_PLCC4_5.0x5.0mm_P3.2mm" H 4450 4750 50  0001 L TNN
 F 3 "https://cdn-shop.adafruit.com/datasheets/WS2812B.pdf" H 4500 4675 50  0001 L TNN
+F 4 "C114586" H 4400 5050 50  0001 C CNN "LCSC"
 	1    4400 5050
 	1    0    0    -1
@@
 F 2 "LED_SMD:LED_WS2812B_PLCC4_5.0x5.0mm_P3.2mm" H 3450 4750 50  0001 L TNN
 F 3 "https://cdn-shop.adafruit.com/datasheets/WS2812B.pdf" H 3500 4675 50  0001 L TNN
+F 4 "C114586" H 3400 5050 50  0001 C CNN "LCSC"
 	1    3400 5050
 	1    0    0    -1
@@
 F 2 "LED_SMD:LED_WS2812B_PLCC4_5.0x5.0mm_P3.2mm" H 5450 4750 50  0001 L TNN
 F 3 "https://cdn-shop.adafruit.com/datasheets/WS2812B.pdf" H 5500 4675 50  0001 L TNN
+F 4 "C114586" H 5400 5050 50  0001 C CNN "LCSC"
 	1    5400 5050
 	1    0    0    -1
@@
 F 2 "LED_SMD:LED_WS2812B_PLCC4_5.0x5.0mm_P3.2mm" H 1450 6050 50  0001 L TNN
 F 3 "https://cdn-shop.adafruit.com/datasheets/WS2812B.pdf" H 1500 5975 50  0001 L TNN
+F 4 "C114586" H 1400 6350 50  0001 C CNN "LCSC"
 	1    1400 6350
 	1    0    0    -1
@@
 F 2 "LED_SMD:LED_WS2812B_PLCC4_5.0x5.0mm_P3.2mm" H 2450 6050 50  0001 L TNN
 F 3 "https://cdn-shop.adafruit.com/datasheets/WS2812B.pdf" H 2500 5975 50  0001 L TNN
+F 4 "C114586" H 2400 6350 50  0001 C CNN "LCSC"
 	1    2400 6350
 	1    0    0    -1
@@
 F 2 "LED_SMD:LED_WS2812B_PLCC4_5.0x5.0mm_P3.2mm" H 4450 6050 50  0001 L TNN
 F 3 "https://cdn-shop.adafruit.com/datasheets/WS2812B.pdf" H 4500 5975 50  0001 L TNN
+F 4 "C114586" H 4400 6350 50  0001 C CNN "LCSC"
 	1    4400 6350
 	1    0    0    -1
@@
 F 2 "LED_SMD:LED_WS2812B_PLCC4_5.0x5.0mm_P3.2mm" H 3450 6050 50  0001 L TNN
 F 3 "https://cdn-shop.adafruit.com/datasheets/WS2812B.pdf" H 3500 5975 50  0001 L TNN
+F 4 "C114586" H 3400 6350 50  0001 C CNN "LCSC"
 	1    3400 6350
 	1    0    0    -1
@@
 F 2 "LED_SMD:LED_WS2812B_PLCC4_5.0x5.0mm_P3.2mm" H 5450 6050 50  0001 L TNN
 F 3 "https://cdn-shop.adafruit.com/datasheets/WS2812B.pdf" H 5500 5975 50  0001 L TNN
+F 4 "C114586" H 5400 6350 50  0001 C CNN "LCSC"
 	1    5400 6350
 	1    0    0    -1
@@
 F 2 "MountingHole:MountingHole_4.3mm_M4" H 5350 1350 50  0001 C CNN
 F 3 "~" H 5350 1350 50  0001 C CNN
+F 4 "" H 5350 1350 50  0001 C CNN "JLCPCB_IGNORE"
 	1    5350 1350
 	1    0    0    -1
@@
 F 2 "Icicle:LedStripPads" H 1750 1100 50  0001 C CNN
 F 3 "" H 1750 1100 50  0001 C CNN
+F 4 "" H 1750 1100 50  0001 C CNN "JLCPCB_IGNORE"
 	1    1750 1100
 	1    0    0    1
@@
 F 2 "Icicle:LedStripPads" H 2650 1100 50  0001 C CNN
 F 3 "" H 2650 1100 50  0001 C CNN
+F 4 "" H 2650 1100 50  0001 C CNN "JLCPCB_IGNORE"
 	1    2650 1100
 	-1   0    0    1
@@
 F 2 "Capacitor_SMD:C_1206_3216Metric" H 8738 1700 50  0001 C CNN
 F 3 "~" H 8700 1850 50  0001 C CNN
+F 4 "C13585" V 8700 1850 50  0001 C CNN "LCSC"
 	1    8700 1850
 	0    1    -1   0

Commit message: Added Correct rotation of LEDs
Parts:
- D1, D10, D11, D12, D13, D14, D15, D16, D17, D18, D19, D2, D20, D3, D4, D5, D6, D7, D8, D9: JLCPCB_CORRECTION (none) -> 0;0;180
Changed lines of the file:
@@
 F 3 "https://cdn-shop.adafruit.com/datasheets/WS2812B.pdf" H 1500 2075 50  0001 L TNN
 F 4 "C114586" H 1400 2450 50  0001 C CNN "LCSC"
+F 5 "0;0;180" H 1400 2450 50  0001 C CNN "JLCPCB_CORRECTION"
 	1    1400 2450
 	1    0    0    -1
@@
 F 3 "https://cdn-shop.adafruit.com/datasheets/WS2812B.pdf" H 2500 2075 50  0001 L TNN
 F 4 "C114586" H 2400 2450 50  0001 C CNN "LCSC"
+F 5 "0;0;180" H 2400 2450 50  0001 C CNN "JLCPCB_CORRECTION"
 	1    2400 2450
 	1    0    0    -1
@@
 F 3 "https://cdn-shop.adafruit.com/datasheets/WS2812B.pdf" H 4500 2075 50  0001 L TNN
 F 4 "C114586" H 4400 2450 50  0001 C CNN "LCSC"
+F 5 "0;0;180" H 4400 2450 50  0001 C CNN "JLCPCB_CORRECTION"
 	1    4400 2450
 	1    0    0    -1
@@
 F 3 "https://cdn-shop.adafruit.com/datasheets/WS2812B.pdf" H 3500 2075 50  0001 L TNN
 F 4 "C114586" H 3400 2450 50  0001 C CNN "LCSC"
+F 5 "0;0;180" H 3400 2450 50  0001 C CNN "JLCPCB_CORRECTION"
 	1    3400 2450
 	1    0    0    -1
@@
 F 3 "https://cdn-shop.adafruit.com/datasheets/WS2812B.pdf" H 5500 2075 50  0001 L TNN
 F 4 "C114586" H 5400 2450 50  0001 C CNN "LCSC"
+F 5 "0;0;180" H 5400 2450 50  0001 C CNN "JLCPCB_CORRECTION"
 	1    5400 2450
 	1    0    0    -1
@@
 F 3 "https://cdn-shop.adafruit.com/datasheets/WS2812B.pdf" H 1500 3375 50  0001 L TNN
 F 4 "C114586" H 1400 3750 50  0001 C CNN "LCSC"
+F 5 "0;0;180" H 1400 3750 50  0001 C CNN "JLCPCB_CORRECTION"
 	1    1400 3750
 	1    0    0    -1
@@
 F 3 "https://cdn-shop.adafruit.com/datasheets/WS2812B.pdf" H 2500 3375 50  0001 L TNN
 F 4 "C114586" H 2400 3750 50  0001 C CNN "LCSC"
+F 5 "0;0;180" H 2400 3750 50  0001 C CNN "JLCPCB_CORRECTION"
 	1    2400 3750
 	1    0    0    -1
@@
 F 3 "https://cdn-shop.adafruit.com/datasheets/WS2812B.pdf" H 4500 3375 50  0001 L TNN
 F 4 "C114586" H 4400 3750 50  0001 C CNN "LCSC"
+F 5 "0;0;180" H 4400 3750 50  0001 C CNN "JLCPCB_CORRECTION"
 	1    4400 3750
 	1    0    0    -1
@@
 F 3 "https://cdn-shop.adafruit.com/datasheets/WS2812B.pdf" H 3500 3375 50  0001 L TNN
 F 4 "C114586" H 3400 3750 50  0001 C CNN "LCSC"
+F 5 "0;0;180" H 3400 3750 50  0001 C CNN "JLCPCB_CORRECTION"
 	1    3400 3750
 	1    0    0    -1
@@
 F 3 "https://cdn-shop.adafruit.com/datasheets/WS2812B.pdf" H 5500 3375 50  0001 L TNN
 F 4 "C114586" H 5400 3750 50  0001 C CNN "LCSC"
+F 5 "0;0;180" H 5400 3750 50  0001 C CNN "JLCPCB_CORRECTION"
 	1    5400 3750
 	1    0    0    -1
@@
 F 3 "https://cdn-shop.adafruit.com/datasheets/WS2812B.pdf" H 1500 4675 50  0001 L TNN
 F 4 "C114586" H 1400 5050 50  0001 C CNN "LCSC"
+F 5 "0;0;180" H 1400 5050 50  0001 C CNN "JLCPCB_CORRECTION"
 	1    1400 5050
 	1    0    0    -1
@@
 F 3 "https://cdn-shop.adafruit.com/datasheets/WS2812B.pdf" H 2500 4675 50  0001 L TNN
 F 4 "C114586" H 2400 5050 50  0001 C CNN "LCSC"
+F 5 "0;0;180" H 2400 5050 50  0001 C CNN "JLCPCB_CORRECTION"
 	1    2400 5050
 	1    0    0    -1
@@
 F 3 "https://cdn-shop.adafruit.com/datasheets/WS2812B.pdf" H 4500 4675 50  0001 L TNN
 F 4 "C114586" H 4400 5050 50  0001 C CNN "LCSC"
+F 5 "0;0;180" H 4400 5050 50  0001 C CNN "JLCPCB_CORRECTION"
 	1    4400 5050
 	1    0    0    -1
@@
 F 3 "https://cdn-shop.adafruit.com/datasheets/WS2812B.pdf" H 3500 4675 50  0001 L TNN
 F 4 "C114586" H 3400 5050 50  0001 C CNN "LCSC"
+F 5 "0;0;180" H 3400 5050 50  0001 C CNN "JLCPCB_CORRECTION"
 	1    3400 5050
 	1    0    0    -1
@@
 F 3 "https://cdn-shop.adafruit.com/datasheets/WS2812B.pdf" H 5500 4675 50  0001 L TNN
 F 4 "C114586" H 5400 5050 50  0001 C CNN "LCSC"
+F 5 "0;0;180" H 5400 5050 50  0001 C CNN "JLCPCB_CORRECTION"
 	1    5400 5050
 	1    0    0    -1
@@
 F 3 "https://cdn-shop.adafruit.com/datasheets/WS2812B.pdf" H 1500 5975 50  0001 L TNN
 F 4 "C114586" H 1400 6350 50  0001 C CNN "LCSC"
+F 5 "0;0;180" H 1400 6350 50  0001 C CNN "JLCPCB_CORRECTION"
 	1    1400 6350
 	1    0    0    -1
@@
 F 3 "https://cdn-shop.adafruit.com/datasheets/WS2812B.pdf" H 2500 5975 50  0001 L TNN
 F 4 "C114586" H 2400 6350 50  0001 C CNN "LCSC"
+F 5 "0;0;180" H 2400 6350 50  0001 C CNN "JLCPCB_CORRECTION"
 	1    2400 6350
 	1    0    0    -1
@@
 F 3 "https://cdn-shop.adafruit.com/datasheets/WS2812B.pdf" H 4500 5975 50  0001 L TNN
 F 4 "C114586" H 4400 6350 50  0001 C CNN "LCSC"
+F 5 "0;0;180" H 4400 6350 50  0001 C CNN "JLCPCB_CORRECTION"
 	1    4400 6350
 	1    0    0    -1
@@
 F 3 "https://cdn-shop.adafruit.com/datasheets/WS2812B.pdf" H 3500 5975 50  0001 L TNN
 F 4 "C114586" H 3400 6350 50  0001 C CNN "LCSC"
+F 5 "0;0;180" H 3400 6350 50  0001 C CNN "JLCPCB_CORRECTION"
 	1    3400 6350
 	1    0    0    -1
@@
 F 3 "https://cdn-shop.adafruit.com/datasheets/WS2812B.pdf" H 5500 5975 50  0001 L TNN
 F 4 "C114586" H 5400 6350 50  0001 C CNN "LCSC"
+F 5 "0;0;180" H 5400 6350 50  0001 C CNN "JLCPCB_CORRECTION"
 	1    5400 6350
 	1    0    0    -1
